File: os-v1.0/os-v1.0.sch (KiCad schematic (older format))
At the start: 53 parts, among them J1 Conn_01x02, J2 Conn_01x04, Q1 2N7002, SW1 SW_Push, SW2 SW_Push, SW3 SW_Push, SW4 SW_Push, SW5 SW_Push, U1 DS3231MZ, U10 MCP1812AT, U11 MCP73831T-2ACI_OT, U2 BMA400, U3 BMP280, U4 GC9A01_IPS_display, U5 USB-OTG, U6 CH340E, U7 ttgo-32-micro, U8 Quectel_L96, U9 TPS2115A_default

Commit message: add power symbols to all power nets
Parts:
- U4: value GC9A01_IPS_display -> GC9A01_IPS_display_SPI
Connections:
- net VBAT renamed +BATT
- net VOUT renamed VDD
Other:
- note added: "POWER NET FLAGS"
- note removed: "POWER FLAGS"
- note removed: "TODO:\nDEFINE SPI PINS"
- moved on the sheet: C5, C6, J1, J2, U10
